File: poub/Poub.kicad_pcb (KiCad board)
At the start: 4 copper layers, 70.2 x 66.5 mm, 25 parts, among them J1 SensorA, J2 SensorB, J3 Conn_01x02, J4 PCI_express_x1, Q1 S8550, U4 HX711

Commit message: final fabrication data
Parts:
- moved J4 9.66 mm to (102.2, 88.5)
Routing:
- net 3.3V: track 72.8 -> 31.4 mm, vias 0 -> 2
- net 5V_local: track 94.9 -> 87.6 mm
- net VBUS: track 33.4 -> 37.5 mm
- net 5V: track 41.7 -> 45.0 mm
- net SCK: track 25.1 -> 27.3 mm
- net DOUT: track 26.6 -> 28.5 mm
- net GND: track 40.0 -> 40.9 mm
Other:
- board size 70.2 x 66.5 mm -> 70.2 x 60 mm
