File: poub/Poub.kicad_sch (KiCad schematic)
At the start: 25 parts, among them J1 Conn_01x04, J2 Conn_01x04, J4 Conn_01x02, Q1 S8550, U3 PCI_express_x1, U4 HX711

Commit message: Add files via upload
correction of some symbols and footprints
Parts:
- removed D1, D2: 1N5819, Diode_THT:D_DO-41_SOD81_P10.16mm_Horizontal, symbol Diode:1N5819
- removed U3: PCI_express_x1, my_library_KiCad:10061913110CLF, symbol New_Library:PCIexpress
- added D1, D2: FM5817-W, DIOM5025X231N, symbol FM5817-W:FM5817-W
- added J4: PCI_express_x1, 10061913110CLF, symbol 10061913-110CLF:10061913-110CLF
- C4, C5: footprint Capacitor_SMD:C_1206_3216Metric -> Capacitor_SMD:C_0805_2012Metric_Pad1.18x1.45mm_HandSolder; Mfr. No C1206C104J4GACTU -> C0805C104J4RACAUTO
- J1, J2: footprint TerminalBlock:TerminalBlock_MaiXu_MX126-5.0-04P_1x04_P5.00mm -> TerminalBlock:TerminalBlock_Xinya_XY308-2.54-4P_1x04_P2.54mm_Horizontal; Mfr. No 691137910004 -> 1725672
- J3: renamed from J4; footprint TerminalBlock:TerminalBlock_MaiXu_MX126-5.0-02P_1x02_P5.00mm -> TerminalBlock:TerminalBlock_Xinya_XY308-2.54-2P_1x02_P2.54mm_Horizontal; Mfr. No 691137910004 -> 1725656
- Q1: footprint Package_TO_SOT_THT:TO-92_Inline -> Package_TO_SOT_SMD:SOT-23-3
Connections:
- net 3.3V: now also J4.A17, J4.B17
- net 5V: now also D1.1 (K), D2.1 (K)
- net 5V_local: now also D1.2 (A), J4.A18, J4.B18
- net DOUT: now also J4.A1
- net GND: now also J4.A12, J4.A14, J4.A16, J4.A6, J4.A7, J4.A8, J4.A9, J4.B12, J4.B14, J4.B16, J4.B6, J4.B9
- net SCK: now also J4.A2
- net VBUS: now also D2.2 (A), J4.A15, J4.B15

Commit message: final fabrication data
Parts:
- D1, D2: Mfr. No (none) -> FM5817-W; Mouser Part Number 583-FM5817 -> (none)
- U1: Mfr. No TSR0.5-2450 -> TSR 0.5-2450
- U4: now left out of the parts list
Changed lines of the file:
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@@
 			)
 		)
-		(property "Mouser Part Number" "583-FM5817"
+		(property "Mouser Part Number" ""
 			(at 106.68 653.67 0)
 			(effects
@@
 			)
 		)
+		(property "Mfr. No" "FM5817-W"
+			(at 119.38 160.02 0)
+			(effects
+				(font
+					(size 1.27 1.27)
+				)
+				(hide yes)
+			)
+		)
 		(pin "2"
 		)
@@
 			)
 		)
-		(property "Mfr. No" "TSR0.5-2450"
+		(property "Mfr. No" "TSR 0.5-2450"
 			(at 55.88 37.084 0)
 			(effects
@@
 			)
 		)
-		(property "Mouser Part Number" "583-FM5817"
+		(property "Mouser Part Number" ""
 			(at 106.68 640.97 0)
 			(effects
@@
 					(size 1.27 1.27)
 				)
+			)
+		)
+		(property "Mfr. No" "FM5817-W"
+			(at 119.38 147.32 0)
+			(effects
+				(font
+					(size 1.27 1.27)
+				)
+				(hide yes)
 			)
 		)
@@
 		(unit 1)
 		(exclude_from_sim no)
-		(in_bom yes)
-		(on_board yes)
-		(dnp no)
+		(in_bom no)
+		(on_board yes)
+		(dnp no)
